Commit message: simulation_works

File: laracna/urdf/laracna.urdf (robot description, URDF)
Before this commit: robot laracna, 13 links, 12 joints
Links:
- link base_link: geometry collision mesh filename=package://laracna/meshes/base_link.stl; visual mesh filename=package://laracna/meshes/base_link.stl
- link coxa_lb: geometry collision mesh filename=package://laracna/meshes/coxa_lb.stl; visual mesh filename=package://laracna/meshes/coxa_lb.stl
- link coxa_lt: geometry collision mesh filename=package://laracna/meshes/coxa_lt.stl; visual mesh filename=package://laracna/meshes/coxa_lt.stl
- link coxa_rb: geometry collision mesh filename=package://laracna/meshes/coxa_rb.stl; visual mesh filename=package://laracna/meshes/coxa_rb.stl
- link coxa_rt: geometry collision mesh filename=package://laracna/meshes/coxa_rt.stl; visual mesh filename=package://laracna/meshes/coxa_rt.stl
- link femur_lb: geometry collision mesh filename=package://laracna/meshes/femur_lb.stl; visual mesh filename=package://laracna/meshes/femur_lb.stl
- link femur_lt: geometry collision mesh filename=package://laracna/meshes/femur_lt.stl; visual mesh filename=package://laracna/meshes/femur_lt.stl
- link femur_rb: geometry collision mesh filename=package://laracna/meshes/femur_rb.stl; visual mesh filename=package://laracna/meshes/femur_rb.stl
- link femur_rt: geometry collision mesh filename=package://laracna/meshes/femur_rt.stl; visual mesh filename=package://laracna/meshes/femur_rt.stl
- link tibia_lb: geometry collision mesh filename=package://laracna/meshes/tibia_lb.stl; visual mesh filename=package://laracna/meshes/tibia_lb.stl
- link tibia_lt: geometry collision mesh filename=package://laracna/meshes/tibia_lt.stl; visual mesh filename=package://laracna/meshes/tibia_lt.stl
- link tibia_rb: geometry collision mesh filename=package://laracna/meshes/tibia_rb.stl; visual mesh filename=package://laracna/meshes/tibia_rb.stl
- link tibia_rt: geometry collision mesh filename=package://laracna/meshes/tibia_rt.stl; visual mesh filename=package://laracna/meshes/tibia_rt.stl

File: laracna_sim/urdf/laracna.urdf (robot description, URDF)
Before this commit: robot laracna, 13 links, 12 joints
Links:
- link base_link: geometry collision mesh filename=/home/ale/laracna_ws/src/laracna_sim/meshes/base_link.stl; visual mesh filename=/home/ale/laracna_ws/src/laracna_sim/meshes/base_link.stl
- link coxa_lb: geometry collision mesh filename=/home/ale/laracna_ws/src/laracna_sim/meshes/coxa_lb.stl; visual mesh filename=/home/ale/laracna_ws/src/laracna_sim/meshes/coxa_lb.stl
- link coxa_lt: geometry collision mesh filename=/home/ale/laracna_ws/src/laracna_sim/meshes/coxa_lt.stl; visual mesh filename=/home/ale/laracna_ws/src/laracna_sim/meshes/coxa_lt.stl
- link coxa_rb: geometry collision mesh filename=/home/ale/laracna_ws/src/laracna_sim/meshes/coxa_rb.stl; visual mesh filename=/home/ale/laracna_ws/src/laracna_sim/meshes/coxa_rb.stl
- link coxa_rt: geometry collision mesh filename=/home/ale/laracna_ws/src/laracna_sim/meshes/coxa_rt.stl; visual mesh filename=/home/ale/laracna_ws/src/laracna_sim/meshes/coxa_rt.stl
- link femur_lb: geometry collision mesh filename=/home/ale/laracna_ws/src/laracna_sim/meshes/femur_lb.stl; visual mesh filename=/home/ale/laracna_ws/src/laracna_sim/meshes/femur_lb.stl
- link femur_lt: geometry collision mesh filename=/home/ale/laracna_ws/src/laracna_sim/meshes/femur_lt.stl; visual mesh filename=/home/ale/laracna_ws/src/laracna_sim/meshes/femur_lt.stl
- link femur_rb: geometry collision mesh filename=/home/ale/laracna_ws/src/laracna_sim/meshes/femur_rb.stl; visual mesh filename=/home/ale/laracna_ws/src/laracna_sim/meshes/femur_rb.stl
- link femur_rt: geometry collision mesh filename=/home/ale/laracna_ws/src/laracna_sim/meshes/femur_rt.stl; visual mesh filename=/home/ale/laracna_ws/src/laracna_sim/meshes/femur_rt.stl
- link tibia_lb: geometry collision mesh filename=/home/ale/laracna_ws/src/laracna_sim/meshes/tibia_lb.stl; visual mesh filename=/home/ale/laracna_ws/src/laracna_sim/meshes/tibia_lb.stl
- link tibia_lt: geometry collision mesh filename=/home/ale/laracna_ws/src/laracna_sim/meshes/tibia_lt.stl; visual mesh filename=/home/ale/laracna_ws/src/laracna_sim/meshes/tibia_lt.stl
- link tibia_rb: geometry collision mesh filename=/home/ale/laracna_ws/src/laracna_sim/meshes/tibia_rb.stl; visual mesh filename=/home/ale/laracna_ws/src/laracna_sim/meshes/tibia_rb.stl
- link tibia_rt: geometry collision mesh filename=/home/ale/laracna_ws/src/laracna_sim/meshes/tibia_rt.stl; visual mesh filename=/home/ale/laracna_ws/src/laracna_sim/meshes/tibia_rt.stl
